File: BitConnector.sch (KiCad schematic (older format))
At the start: 14 parts, among them J1 JTAG, SW1 reset, U1 XC95##XL-VQ44

Commit message: Introduce BitConnector_v4X     - Add hardware debouncing via schmitt trigger action     - The Schmnitt Triger adds another external inverter. Usable over J2.     - As an alternative, add jumper to bridge the Schmitt trigger.         Use this if the component is not available.     - Partial redesign of the routing     - Add schematic as PDF now
Parts:
- added C4: 100nF, Capacitor_SMD:C_0603_1608Metric, symbol Device:C
- added J2: Conn_01x02, Connector_PinSocket_2.54mm:PinSocket_1x02_P2.54mm_Vertical, symbol Connector_Generic:Conn_01x02
- added JP1: disable_schmitt_trigger_action, Jumper:SolderJumper-2_P1.3mm_Open_RoundedPad1.0x1.5mm, symbol Jumper:SolderJumper_2_Open
- added R5: 100K, Resistor_SMD:R_0805_2012Metric_Pad1.15x1.40mm_HandSolder, symbol Device:R
- added R7: 10K, Resistor_SMD:R_0805_2012Metric_Pad1.15x1.40mm_HandSolder, symbol Device:R
- added U2: 74LVC2G14, Package_TO_SOT_SMD:SOT-363_SC-70-6_Handsoldering, symbol 74xGxx:74LVC2G14
- R1, R2, R3: value 4K7 -> 10K
- R6: renamed from R5; value 4K7 -> 10K
- U1: symbol BitConnector-rescue:Xilinx_CPLD_VQFP_2_DIP-rescue_XC9536XL-VQ44-Xilinx-VQ44-Xilinx_CPLD_VQFP_2_DIP-rescue-BitConnector -> BitConnector-rescue:Xilinx_CPLD_VQFP_2_DIP-rescue_XC9536XL-VQ44-Xilinx-VQ44-Xilinx_CPLD_VQFP_2_DIP-rescue-BitConnector-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
Connections:
- net +3V3: now also R6.1; no longer SW1.1
- net GND: now also SW1.2, C4.2, R7.2, U2.2 (GND), U2.2 (GND); no longer R6.2
- net VCC: now also U2.5 (VCC), U2.5 (VCC)
- new net: JP1.2 (B), R5.1, R6.2, SW1.1
- new net: JP1.1 (A), U1.33 (I/O/GSR), U2.4
- new net: C4.1, R5.2, U2.3
- new net: J2.1 (Pin_1), R7.1, U2.1
- new net: J2.2 (Pin_2), U2.6
Other:
- moved on the sheet: C1, C2, C3, D1, R1, R2, R3, R4, R6, SW1, U1

Commit message: Change package for 74LVC2G14 from SOT363 to SOT457
Parts:
- U2: footprint Package_TO_SOT_SMD:SOT-363_SC-70-6_Handsoldering -> Package_SO:SC-74-6_1.5x2.9mm_P0.95mm
Changed lines of the file:
@@
 EESchema Schematic File Version 4
-LIBS:BitConnector-cache
 EELAYER 30 0
 EELAYER END
@@
 F 0 "U2" H 5775 1633 50  0000 C CNN
 F 1 "74LVC2G14" H 5775 1724 50  0000 C CNN
-F 2 "Package_TO_SOT_SMD:SOT-363_SC-70-6_Handsoldering" H 5800 1900 50  0001 C CNN
+F 2 "Package_SO:SC-74-6_1.5x2.9mm_P0.95mm" H 5800 1900 50  0001 C CNN
 F 3 "https://www.ti.com/lit/ds/symlink/sn74lvc2g14.pdf" H 5800 1900 50  0001 C CNN
 	1    5800 1900
@@
 F 0 "U2" H 6025 4017 50  0000 C CNN
 F 1 "74LVC2G14" H 6025 3926 50  0000 C CNN
-F 2 "Package_TO_SOT_SMD:SOT-363_SC-70-6_Handsoldering" H 6050 3750 50  0001 C CNN
+F 2 "Package_SO:SC-74-6_1.5x2.9mm_P0.95mm" H 6050 3750 50  0001 C CNN
 F 3 "https://www.ti.com/lit/ds/symlink/sn74lvc2g14.pdf" H 6050 3750 50  0001 C CNN
 	2    6050 3750

Commit message: first attempt of the new v5X version
    details:
    	- switch solder pad for resistors from 1.15mm to 1.20mm
	- add additional 10nF bypass capacitor according to
	  Xilinx XAPP104 (3.0.1) specification
	- Completely new board layout created to improve
	  GND and Vcc connection and suppress interference signals
	- fallback to v3X (minimal configuration) is retained
	- 74LVC2G14 (schmitt trigger) now has a better footprint
Parts:
- added C5, C6, C7: 10nF, Capacitor_SMD:C_0603_1608Metric, symbol Device:C
- R1, R2, R3, R4, R5, R6, R7: footprint Resistor_SMD:R_0805_2012Metric_Pad1.15x1.40mm_HandSolder -> Resistor_SMD:R_0805_2012Metric_Pad1.20x1.40mm_HandSolder
- U1: symbol BitConnector-rescue:Xilinx_CPLD_VQFP_2_DIP-rescue_XC9536XL-VQ44-Xilinx-VQ44-Xilinx_CPLD_VQFP_2_DIP-rescue-BitConnector-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 -> XC96xxxl:Xilinx_CPLD_VQFP_2_DIP-rescue_XC9536XL-VQ44-Xilinx-VQ44-Xilinx_CPLD_VQFP_2_DIP-rescue-BitConnector-BitConnecto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
Connections:
- net +3V3: now also C5.1, C6.1
- net GND: now also C5.2, C6.2, C7.1
- net VCC: now also C7.2
Other:
- moved on the sheet: C1, C3
Changed lines of the file:
@@
 Sheet 1 1
 Title "XC95## VQ44 to DIP 40"
-Date "2019-10-25"
+Date "2021-02-01"
 Rev "v04X"
 Comp ""
@@
 L Device:C C1
 U 1 1 5BE5958E
-P 3200 2050
-F 0 "C1" V 2948 2050 50  0000 C CNN
-F 1 "100nF" V 3039 2050 50  0000 C CNN
-F 2 "Capacitor_SMD:C_0603_1608Metric" H 3238 1900 50  0001 C CNN
-F 3 "~" H 3200 2050 50  0001 C CNN
-	1    3200 2050
+P 3200 1950
+F 0 "C1" V 2948 1950 50  0000 C CNN
+F 1 "100nF" V 3039 1950 50  0000 C CNN
+F 2 "Capacitor_SMD:C_0603_1608Metric" H 3238 1800 50  0001 C CNN
+F 3 "~" H 3200 1950 50  0001 C CNN
+	1    3200 1950
 	0    1    1    0
 $EndComp
@@
 L Device:C C3
 U 1 1 5BE59733
-P 3700 2050
-F 0 "C3" V 3448 2050 50  0000 C CNN
-F 1 "100nF" V 3539 2050 50  0000 C CNN
-F 2 "Capacitor_SMD:C_0603_1608Metric" H 3738 1900 50  0001 C CNN
-F 3 "~" H 3700 2050 50  0001 C CNN
-	1    3700 2050
-	0    1    1    0
-$EndComp
-Wire Wire Line
-	3350 2450 3350 2050
-Wire Wire Line
-	3550 2450 3550 2050
+P 3700 1950
+F 0 "C3" V 3650 2350 50  0000 C CNN
+F 1 "100nF" V 3650 2150 50  0000 C CNN
+F 2 "Capacitor_SMD:C_0603_1608Metric" H 3738 1800 50  0001 C CNN
+F 3 "~" H 3700 1950 50  0001 C CNN
+	1    3700 1950
+	0    1    1    0
+$EndComp
 Wire Wire Line
 	3450 1400 3450 2450
 Wire Wire Line
 	3850 1400 3850 1200
-Wire Wire Line
-	3350 2050 3350 1400
-Connection ~ 3350 2050
-Connection ~ 3550 2050
 $Comp
 L Device:R R3
@@
 F 0 "R3" V 4600 5350 50  0000 C CNN
 F 1 "10K" H 4450 5350 50  0000 C CNN
-F 2 "Resistor_SMD:R_0805_2012Metric_Pad1.15x1.40mm_HandSolder" V 4530 5350 50  0001 C CNN
+F 2 "Resistor_SMD:R_0805_2012Metric_Pad1.20x1.40mm_HandSolder" V 4530 5350 50  0001 C CNN
 F 3 "~" H 4600 5350 50  0001 C CNN
 	1    4600 5350
@@
 F 0 "R1" V 4300 5350 50  0000 C CNN
 F 1 "10K" H 4150 5350 50  0000 C CNN
-F 2 "Resistor_SMD:R_0805_2012Metric_Pad1.15x1.40mm_HandSolder" V 4230 5350 50  0001 C CNN
+F 2 "Resistor_SMD:R_0805_2012Metric_Pad1.20x1.40mm_HandSolder" V 4230 5350 50  0001 C CNN
 F 3 "~" H 4300 5350 50  0001 C CNN
 	1    4300 5350
@@
 F 0 "R2" V 4450 5350 50  0000 C CNN
 F 1 "10K" H 4450 5550 50  0000 C TNN
-F 2 "Resistor_SMD:R_0805_2012Metric_Pad1.15x1.40mm_HandSolder" V 4380 5350 50  0001 C CNN
+F 2 "Resistor_SMD:R_0805_2012Metric_Pad1.20x1.40mm_HandSolder" V 4380 5350 50  0001 C CNN
 F 3 "~" H 4450 5350 50  0001 C CNN
 	1    4450 5350
@@
 Wire Wire Line
 	4150 3850 4550 3850
-Text Label 3550 2250 0    50   ~ 0
+Text Label 3600 850  0    50   ~ 0
 VCCIO
 Wire Wire Line
-	3050 2050 2950 2050
-Wire Wire Line
-	3850 2050 4000 2050
+	3050 2300 2950 2300
+Wire Wire Line
+	3850 2300 4000 2300
 Wire Wire Line
 	4600 4750 4700 4750
@@
 L power:GND #PWR06
 U 1 1 5C4B7825
-P 4000 2050
-F 0 "#PWR06" H 4000 1800 50  0001 C CNN
-F 1 "GND" H 4005 1877 50  0000 C CNN
-F 2 "" H 4000 2050 50  0001 C CNN
-F 3 "" H 4000 2050 50  0001 C CNN
-	1    4000 2050
+P 4000 2300
+F 0 "#PWR06" H 4000 2050 50  0001 C CNN
+F 1 "GND" H 4005 2127 50  0000 C CNN
+F 2 "" H 4000 2300 50  0001 C CNN
+F 3 "" H 4000 2300 50  0001 C CNN
+	1    4000 2300
 	1    0    0    -1
 $EndComp
@@
 L power:GND #PWR01
 U 1 1 5C4B78B2
-P 2950 2050
-F 0 "#PWR01" H 2950 1800 50  0001 C CNN
-F 1 "GND" H 2955 1877 50  0000 C CNN
-F 2 "" H 2950 2050 50  0001 C CNN
-F 3 "" H 2950 2050 50  0001 C CNN
-	1    2950 2050
+P 2950 2300
+F 0 "#PWR01" H 2950 2050 50  0001 C CNN
+F 1 "GND" H 2955 2127 50  0000 C CNN
+F 2 "" H 2950 2300 50  0001 C CNN
+F 3 "" H 2950 2300 50  0001 C CNN
+	1    2950 2300
 	1    0    0    -1
 $EndComp
@@
 GP_IO_33
 $Comp
-L BitConnector-rescue:Xilinx_CPLD_VQFP_2_DIP-rescue_XC9536XL-VQ44-Xilinx-VQ44-Xilinx_CPLD_VQFP_2_DIP-rescue-BitConnector-BitConnector-rescue U1
+L XC96xxxl:Xilinx_CPLD_VQFP_2_DIP-rescue_XC9536XL-VQ44-Xilinx-VQ44-Xilinx_CPLD_VQFP_2_DIP-rescue-BitConnector-BitConnector-rescue-BitConnector-rescue U1
 U 1 1 5C7597D2
 P 3450 3850
-F 0 "U1" H 3450 5428 50  0000 C CNN
-F 1 "XC95##XL-VQ44" H 3450 5337 50  0000 C CNN
+F 0 "U1" H 3450 4550 50  0000 C CNN
+F 1 "XC95##XL-VQ44" H 3450 4450 50  0000 C CNN
 F 2 "Package_QFP:LQFP-44_10x10mm_P0.8mm" H 3450 3850 50  0001 C CNN
 F 3 "xilinx/xc9536.pdf" H 3450 3850 50  0001 C CNN
@@
 F 0 "R4" V 5000 5600 50  0000 C CNN
 F 1 "120" H 4850 5600 50  0000 C CNN
-F 2 "Resistor_SMD:R_0805_2012Metric_Pad1.15x1.40mm_HandSolder" V 4930 5600 50  0001 C CNN
+F 2 "Resistor_SMD:R_0805_2012Metric_Pad1.20x1.40mm_HandSolder" V 4930 5600 50  0001 C CNN
 F 3 "~" H 5000 5600 50  0001 C CNN
 	1    5000 5600
@@
 $EndComp
 Wire Wire Line
-	3550 5250 3450 5250
-Wire Wire Line
-	3350 5250 3450 5250
-Connection ~ 3350 5250
-Connection ~ 3450 5250
-Wire Wire Line
 	7050 3250 7050 3350
 $Comp
@@
 F 0 "R6" V 7050 3500 50  0000 C CNN
 F 1 "10K" H 6900 3500 50  0000 C CNN
-F 2 "Resistor_SMD:R_0805_2012Metric_Pad1.15x1.40mm_HandSolder" V 6980 3500 50  0001 C CNN
+F 2 "Resistor_SMD:R_0805_2012Metric_Pad1.20x1.40mm_HandSolder" V 6980 3500 50  0001 C CNN
 F 3 "~" H 7050 3500 50  0001 C CNN
 	1    7050 3500
@@
 F 0 "R7" V 6300 2150 50  0000 C CNN
 F 1 "10K" H 6150 2150 50  0000 C CNN
-F 2 "Resistor_SMD:R_0805_2012Metric_Pad1.15x1.40mm_HandSolder" V 6230 2150 50  0001 C CNN
+F 2 "Resistor_SMD:R_0805_2012Metric_Pad1.20x1.40mm_HandSolder" V 6230 2150 50  0001 C CNN
 F 3 "~" H 6300 2150 50  0001 C CNN
 	1    6300 2150
@@
 F 0 "R5" V 6650 3750 50  0000 C CNN
 F 1 "100K" H 6500 3750 50  0000 C CNN
-F 2 "Resistor_SMD:R_0805_2012Metric_Pad1.15x1.40mm_HandSolder" V 6580 3750 50  0001 C CNN
+F 2 "Resistor_SMD:R_0805_2012Metric_Pad1.20x1.40mm_HandSolder" V 6580 3750 50  0001 C CNN
 F 3 "~" H 6650 3750 50  0001 C CNN
 	1    6650 3750
@@
 P 3550 1700
 F 0 "#FLG0102" H 3550 1775 50  0001 C CNN
-F 1 "PWR_FLAG" V 3550 1828 50  0000 L CNN
+F 1 "PWR_FLAG" V 3550 1850 50  0000 L CNN
 F 2 "" H 3550 1700 50  0001 C CNN
 F 3 "~" H 3550 1700 50  0001 C CNN
@@
 Wire Wire Line
 	3550 1650 3550 1700
-Wire Wire Line
-	3550 1700 3550 2050
 Connection ~ 3550 1700
 $Comp
@@
 P 3450 1100
 F 0 "#FLG0103" H 3450 1175 50  0001 C CNN
-F 1 "PWR_FLAG" V 3450 1227 50  0000 L CNN
+F 1 "PWR_FLAG" V 3550 1200 50  0000 L CNN
 F 2 "" H 3450 1100 50  0001 C CNN
 F 3 "~" H 3450 1100 50  0001 C CNN
@@
 Wire Wire Line
 	6300 2300 6300 2400
+Wire Wire Line
+	3550 5250 3450 5250
+Wire Wire Line
+	3450 5250 3350 5250
+Connection ~ 3450 5250
+Connection ~ 3350 5250
+Wire Wire Line
+	3550 1700 3550 1950
+Connection ~ 3550 1950
+Wire Wire Line
+	3550 1950 3550 2300
+$Comp
+L Device:C C7
+U 1 1 60208479
+P 3700 2300
+F 0 "C7" V 3550 2500 50  0000 C CNN
+F 1 "10nF" V 3539 2300 50  0000 C CNN
+F 2 "Capacitor_SMD:C_0603_1608Metric" H 3738 2150 50  0001 C CNN
+F 3 "~" H 3700 2300 50  0001 C CNN
+	1    3700 2300
+	0    1    1    0
+$EndComp
+Text Label 3600 2550 0    50   ~ 0
+VCCIO
+Connection ~ 3550 2300
+Wire Wire Line
+	3550 2300 3550 2450
+Wire Wire Line
+	3850 1950 3850 2300
+Connection ~ 3850 2300
+Connection ~ 3350 1950
+Wire Wire Line
+	3350 1950 3350 1400
+Wire Wire Line
+	3350 1950 3350 2300
+$Comp
+L Device:C C6
+U 1 1 6021F022
+P 3200 2300
+F 0 "C6" V 3050 2050 50  0000 C CNN
+F 1 "10nF" V 3039 2300 50  0000 C CNN
+F 2 "Capacitor_SMD:C_0603_1608Metric" H 3238 2150 50  0001 C CNN
+F 3 "~" H 3200 2300 50  0001 C CNN
+	1    3200 2300
+	0    1    1    0
+$EndComp
+Text Label 3050 2550 0    50   ~ 0
+VCCIO
+Wire Wire Line
+	3050 1950 3050 2300
+Connection ~ 3050 2300
+$Comp
+L Device:C C5
+U 1 1 602344F2
+P 3200 1400
+F 0 "C5" V 2950 1400 50  0000 C CNN
+F 1 "10nF" V 3039 1400 50  0000 C CNN
+F 2 "Capacitor_SMD:C_0603_1608Metric" H 3238 1250 50  0001 C CNN
+F 3 "~" H 3200 1400 50  0001 C CNN
+	1    3200 1400
+	0    1    1    0
+$EndComp
+Wire Wire Line
+	3050 1400 3050 1600
+$Comp
+L power:GND #PWR08
+U 1 1 602399DD
+P 3050 1600
+F 0 "#PWR08" H 3050 1350 50  0001 C CNN
+F 1 "GND" H 2950 1450 50  0000 C CNN
+F 2 "" H 3050 1600 50  0001 C CNN
+F 3 "" H 3050 1600 50  0001 C CNN
+	1    3050 1600
+	1    0    0    -1
+$EndComp
+Connection ~ 3350 2300
+Wire Wire Line
+	3350 2300 3350 2450
 $EndSCHEMATC
